File: KiCad/DriverStage.kicad_sch (KiCad schematic)
At the start: 21 parts, among them CN201 MR60-F, U201 DRV8323HRTAT

Commit message: mostly finished routing
Connections:
- net VREF is gone; now on net +3.3V: C205.1, U201.24 (VREF)
- net at C203.1: now also U201.2 (CPH); no longer U201.1 (CPL)
- net at C203.2: now also U201.1 (CPL); no longer U201.2 (CPH)
- net 3.3V renamed +3.3V
Other:
- moved on the sheet: C203
Changed lines of the file:
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@@
+	(wire
+		(pts
+			(xy 265.43 40.64) (xy 275.59 40.64)
+		)
+		(stroke
+			(width 0)
+			(type default)
+		)
+	)
 	(wire
 		(pts
@@
 			(width 0)
 			(type default)
+		)
+	)
+	(label "VREF"
+		(at 265.43 40.64 0)
+		(effects
+			(font
+				(size 1.27 1.27)
+			)
+			(justify left bottom)
 		)
 	)
@@
 	)
 	(symbol
+		(lib_id "power:+3.3V")
+		(at 275.59 53.34 0)
+		(unit 1)
+		(body_style 1)
+		(exclude_from_sim no)
+		(in_bom yes)
+		(on_board yes)
+		(in_pos_files yes)
+		(dnp no)
+		(fields_autoplaced yes)
+		(property "Reference" "#PWR0211"
+			(at 275.59 57.15 0)
+			(hide yes)
+			(show_name no)
+			(do_not_autoplace no)
+			(effects
+				(font
+					(size 1.27 1.27)
+				)
+			)
+		)
+		(property "Value" "+3.3V"
+			(at 275.59 48.26 0)
+			(show_name no)
+			(do_not_autoplace no)
+			(effects
+				(font
+					(size 1.27 1.27)
+				)
+			)
+		)
+		(property "Footprint" ""
+			(at 275.59 53.34 0)
+			(hide yes)
+			(show_name no)
+			(do_not_autoplace no)
+			(effects
+				(font
+					(size 1.27 1.27)
+				)
+			)
+		)
+		(property "Datasheet" ""
+			(at 275.59 53.34 0)
+			(hide yes)
+			(show_name no)
+			(do_not_autoplace no)
+			(effects
+				(font
+					(size 1.27 1.27)
+				)
+			)
+		)
+		(property "Description" "Power symbol creates a global label with name \"+3.3V\""
+			(at 275.59 53.34 0)
+			(hide yes)
+			(show_name no)
+			(do_not_autoplace no)
+			(effects
+				(font
+					(size 1.27 1.27)
+				)
+			)
+		)
+		(pin "1"
+		)
+		(instances
+			(project "simpleFOC Dual Motor Controller"
+				(path "/0dffc378-5905-459a-b0cb-e8e514a8bbef/de390f81-41fc-4236-a904-44260774a171"
+					(reference "#PWR0211")
+					(unit 1)
+				)
+				(path "/0dffc378-5905-459a-b0cb-e8e514a8bbef/f2c2b770-272c-4740-ba73-c3bb2a232079"
+					(reference "#PWR0602")
+					(unit 1)
+				)
+			)
+		)
+	)
+	(symbol
 		(lib_id "power:GNDA")
 		(at 44.45 134.62 0)
@@
 	(symbol
 		(lib_id "Device:C_Small")
-		(at 101.6 140.97 90)
+		(at 101.6 140.97 270)
+		(mirror x)
 		(unit 1)
 		(body_style 1)
@@
 		(in_pos_files yes)
 		(dnp no)
-		(fields_autoplaced yes)
 		(property "Reference" "C203"
-			(at 101.6063 134.62 90)
+			(at 101.5937 134.62 90)
 			(show_name no)
 			(do_not_autoplace no)
@@
 		)
 		(property "Value" "47n"
-			(at 101.6063 137.16 90)
+			(at 101.5937 137.16 90)
 			(show_name no)
 			(do_not_autoplace no)
@@
 	)
 	(symbol
-		(lib_id "PCM_SparkFun-PowerSymbol:3.3V")
-		(at 275.59 53.34 0)
-		(unit 1)
-		(body_style 1)
-		(exclude_from_sim no)
-		(in_bom yes)
-		(on_board yes)
-		(in_pos_files yes)
-		(dnp no)
-		(fields_autoplaced yes)
-		(property "Reference" "#PWR0211"
-			(at 275.59 57.15 0)
-			(hide yes)
-			(show_name no)
-			(do_not_autoplace no)
-			(effects
-				(font
-					(size 1.27 1.27)
-				)
-			)
-		)
-		(property "Value" "3.3V"
-			(at 275.59 49.53 0)
-			(show_name no)
-			(do_not_autoplace yes)
-			(effects
-				(font
-					(size 1.27 1.27)
-				)
-			)
-		)
-		(property "Footprint" ""
-			(at 275.59 53.34 0)
-			(hide yes)
-			(show_name no)
-			(do_not_autoplace no)
-			(effects
-				(font
-					(size 1.27 1.27)
-				)
-			)
-		)
-		(property "Datasheet" ""
-			(at 275.59 53.34 0)
-			(hide yes)
-			(show_name no)
-			(do_not_autoplace no)
-			(effects
-				(font
-					(size 1.27 1.27)
-				)
-			)
-		)
-		(property "Description" "Power symbol creates a global label with name \"3.3V\""
-			(at 275.59 59.69 0)
-			(hide yes)
-			(show_name no)
-			(do_not_autoplace no)
-			(effects
-				(font
-					(size 1.27 1.27)
-				)
-			)
-		)
-		(pin "1"
-		)
-		(instances
-			(project "simpleFOC Dual Motor Controller"
-				(path "/0dffc378-5905-459a-b0cb-e8e514a8bbef/de390f81-41fc-4236-a904-44260774a171"
-					(reference "#PWR0211")
-					(unit 1)
-				)
-				(path "/0dffc378-5905-459a-b0cb-e8e514a8bbef/f2c2b770-272c-4740-ba73-c3bb2a232079"
-					(reference "#PWR0222")
-					(unit 1)
-				)
-			)
-		)
-	)
-	(symbol
 		(lib_id "Device:C_Small")
 		(at 50.8 57.15 0)
@@
 					(unit 1)
 				)
+			)
+		)
+	)
+	(symbol
+		(lib_id "power:+3.3V")
+		(at 275.59 40.64 0)
+		(unit 1)
+		(body_style 1)
+		(exclude_from_sim no)
+		(in_bom yes)
+		(on_board yes)
+		(in_pos_files yes)
+		(dnp no)
+		(fields_autoplaced yes)
+		(property "Reference" "#PWR0222"
+			(at 275.59 44.45 0)
+			(hide yes)
+			(show_name no)
+			(do_not_autoplace no)
+			(effects
+				(font
+					(size 1.27 1.27)
+				)
+			)
+		)
+		(property "Value" "+3.3V"
+			(at 275.59 35.56 0)
+			(show_name no)
+			(do_not_autoplace no)
+			(effects
+				(font
+					(size 1.27 1.27)
+				)
+			)
+		)
+		(property "Footprint" ""
+			(at 275.59 40.64 0)
+			(hide yes)
+			(show_name no)
+			(do_not_autoplace no)
+			(effects
+				(font
+					(size 1.27 1.27)
+				)
+			)
+		)
+		(property "Datasheet" ""
+			(at 275.59 40.64 0)
+			(hide yes)
+			(show_name no)
+			(do_not_autoplace no)
+			(effects
+				(font
+					(size 1.27 1.27)
+				)
+			)
+		)
+		(property "Description" "Power symbol creates a global label with name \"+3.3V\""
+			(at 275.59 40.64 0)
+			(hide yes)
+			(show_name no)
+			(do_not_autoplace no)
+			(effects
+				(font
+					(size 1.27 1.27)
+				)
+			)
+		)
+		(pin "1"
+		)
+		(instances
+			(project "simpleFOC Dual Motor Controller"
+				(path "/0dffc378-5905-459a-b0cb-e8e514a8bbef/de390f81-41fc-4236-a904-44260774a171"
+					(reference "#PWR0222")
+					(unit 1)
+				)
+				(path "/0dffc378-5905-459a-b0cb-e8e514a8bbef/f2c2b770-272c-4740-ba73-c3bb2a232079"
+					(reference "#PWR0603")
+					(unit 1)
+				)

Commit message: finished iteration 1
Parts:
- removed R224: 47k, Resistor_SMD:R_0402_1005Metric, symbol Device:R_Small
- added R207, R208: 100k, Resistor_SMD:R_0402_1005Metric, symbol Device:R_Small
- C201: footprint Capacitor_SMD:C_0805_2012Metric -> Capacitor_SMD:C_0402_1005Metric
- C205: value 0.1u -> 100n
Connections:
- net +3.3V: no longer C205.1, U201.24 (VREF)
- net GND: now also U201.26 (MODE), R207.2, R208.2
- net ~{HI-Z} renamed INLA
- net INLA: no longer U201.37 (INLB), U201.39 (INLC)
- new net INLB: R207.1, U201.37 (INLB)
- new net INLC: R208.1, U201.39 (INLC)
- new net VREF: C205.1, U201.24 (VREF)
Other:
- note added: "IDRIVE: Mosfet Drive Current Target: 300ns Rise, 100ns Fall Gate-Drain Charge: 7.9nC Rise: 7.9nC / 300ns = 30mA -> 18kΩ to AGND Fall: 7.9nC / 150ns = 60mA -> 18kΩ to AGND MODE: PWM input mode 6-PWM -> Mode 0 -> Tie to AGND GAIN: Current Sense Gain 20 V/V -> 47k to GND 40 V/V -> Pull-Up 5 V/V -> Pull-Dowm VDS: Overcurrent Protection Max Current > 35A RDSon@100°C = 0.00516Ω Overcurrent Voltage = 35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"
- note removed: "IDRIVE: Mosfet Drive Current Target: 300ns Rise, 100ns Fall Gate-Drain Charge: 7.9nC Rise: 7.9nC / 300ns = 30mA -> 18kΩ to AGND Fall: 7.9nC / 150ns = 60mA -> 18kΩ to AGND MODE: PWM input mode 3-PWM -> Mode 1 -> 47kΩ to AGND GAIN: Current Sense Gain 20 V/V -> 47k to GND 40 V/V -> Pull-Up 5 V/V -> Pull-Dowm VDS: Overcurrent Protection Max Current > 35A RDSon@100°C = 0.00516Ω Overcurrent Voltage = 3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"
- moved on the sheet: R209, R210
