File: KiCad/simpleFOC Dual Motor Controller.kicad_pcb (KiCad board)
At the start: 4 copper layers, 50 x 50 mm, 100 parts, among them CN201 MR60-F, CN202 MR60-F, J101 Conn_01x04, J102 USB_C_Receptacle_USB2.0_14P, J103 Conn_01x05_2.0mm, J105 Conn_01x05_2.0mm, Q101 AGM6014AP, Q102 AGM6014AP, Q103 AGM6014AP, Q104 AGM6014AP, Q105 AGM6014AP, Q106 AGM6014AP, Q301 AGM6014AP, Q303 AGM6014AP, Q401 AGM6014AP, Q403 AGM6014AP, Q501 AGM6014AP, Q503 AGM6014AP, SW101 TS-1088-AR02016, U101 XC6206P332MR, U102 XT60H-M, U103 ESP32-S3-WROOM-1, U201 DRV8323HRTAT, U202 DRV8323HRTAT

Commit message: started routing
Parts:
- removed the R108 at (87.3, 45.5)
- C105: footprint Capacitor_SMD:C_01005_0402Metric -> Capacitor_SMD:C_0402_1005Metric
- J101: footprint PCM_SparkFun-Connector:JST_1x04_P2.0mm_Vertical_PTH -> Connector_JST:JST_PH_B4B-PH-K_1x04_P2.00mm_Vertical
- R108: footprint Resistor_THT:R_Axial_DIN0204_L3.6mm_D1.6mm_P1.90mm_Vertical -> Resistor_SMD:R_0402_1005Metric
- moved J105 39.6 mm to (81.7, 51.5)
- moved J103 31.3 mm to (82.4, 57.0), turned to -90 degrees
- moved U101 30.7 mm to (82.4, 75.9), turned to 180 degrees
- moved J102 29.2 mm to (92.8, 81.5), turned to 90 degrees
- moved D105 25.8 mm to (87.2, 81.2)
- moved R108 25.7 mm to (87.3, 78.9), turned to 90 degrees
- moved C105 25.7 mm to (84.0, 74.5), turned to 90 degrees
- moved SW101 24.4 mm to (144.0, 71.9), turned to -90 degrees
- moved D106 23.5 mm to (87.2, 80.5)
- moved D102 23.3 mm to (86.2, 76.2), turned to 180 degrees
- moved R107 23.2 mm to (86.3, 78.9), turned to 90 degrees
- moved D107 19.1 mm to (86.2, 74.6), turned to 180 degrees
- moved D104 17.0 mm to (88.5, 73.2), turned to 90 degrees
- moved U102 16.6 mm to (162.4, 64.7)
- moved J101 12.4 mm to (92.8, 67.3), turned to -90 degrees
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Connections:
- U103 pad 10: /snsB2 -> /snsB1
- U103 pad 11: /snsC2 -> /snsA1
- U103 pad 12: /EN2 -> /CAL1
- U103 pad 15: unconnected-(U103-IO3-Pad15) -> /sns_sck
- U103 pad 18: /FAULT2 -> /CHB1
- U103 pad 19: /GAIN2 -> /GAIN1
- U103 pad 22: /sns_sck -> /snsC2
- U103 pad 28: /FAULT1 -> /CHC2
- U103 pad 29: /GAIN1 -> /CHB2
- U103 pad 30: unconnected-(U103-IO37-Pad30) -> /CHA2
- U103 pad 31: /CAL1 -> /CAL2
- U103 pad 32: /EN1 -> /EN2
- U103 pad 33: /CHC1 -> /GAIN2
- U103 pad 34: /CHB1 -> /FAULT2
- U103 pad 38: /snsB1 -> /snsB2
- U103 pad 39: /snsA1 -> /snsA2
- U103 pad 5: /CHA2 -> unconnected-(U103-IO5-Pad5)
- U103 pad 6: /CHB2 -> /CHC1
- U103 pad 7: /CHC2 -> /FAULT1
- U103 pad 8: /CAL2 -> /EN1
- U103 pad 9: /snsA2 -> unconnected-(U103-IO16-Pad9)
Routing:
- net /snsA2: track 0.00 -> 29.3 mm, vias 0 -> 2
- net /snsB2: track 0.00 -> 27.7 mm, vias 0 -> 2
- net /FAULT2: track 1.27 -> 25.5 mm, vias 0 -> 2
- net /snsC2: track 0.00 -> 23.6 mm, vias 0 -> 2
- net /GAIN2: track 3.09 -> 22.6 mm
- net /EN2: track 1.09 -> 19.0 mm
- net /CAL2: track 3.16 -> 16.5 mm
- net Net-(D102-A): track 0.00 -> 11.0 mm
- net /CHA2: track 2.34 -> 12.0 mm
- net /CHB2: track 2.33 -> 10.4 mm
- net /CHC2: track 1.29 -> 7.28 mm
- net /D-: track 0.00 -> 5.04 mm, vias 0 -> 1
- net /D+: track 0.00 -> 4.73 mm, vias 0 -> 1
- net Net-(D104-K): track 4.56 -> 0.00 mm
- net Net-(J102-CC1): track 0.00 -> 4.41 mm, vias 0 -> 2
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- added copper zone on F.Cu, net +5V

Commit message: mostly finished routing
Parts:
- removed D104: SMF5.0A_C19077497, easyeda2kicad:SOD-123FL_L2.7-W1.8-LS3.8-RD
- removed J105: Conn_01x05_2.0mm, Connector_JST:JST_PH_B5B-PH-K_1x05_P2.00mm_Vertical
- added C101: 220u, easyeda2kicad:CAP-TH_BD8.0-P3.50-D0.6-FD, F.Cu at (104.1, 51.7)
- added J104: Conn_01x06, Connector_JST:JST_PH_B6B-PH-K_1x06_P2.00mm_Vertical, F.Cu at (116.7, 62.6)
- added R110: 100k, Resistor_SMD:R_0402_1005Metric, F.Cu at (109.4, 59.7)
- added R111: 100k, Resistor_SMD:R_0402_1005Metric, F.Cu at (109.4, 58.7)
- added U104: H5VND5UB, easyeda2kicad:SOD-523F_L1.7-W0.9-LS1.7-RD, F.Cu at (146.1, 56.3)
- C103: footprint Capacitor_SMD:C_01005_0402Metric -> Capacitor_SMD:C_0402_1005Metric
- C104: footprint Capacitor_SMD:C_1206_3216Metric -> Capacitor_SMD:C_0603_1608Metric
- C111: value C_Small -> 1u; footprint Capacitor_SMD:C_01005_0402Metric -> Capacitor_SMD:C_0402_1005Metric
- J103: value Conn_01x05_2.0mm -> Conn_01x06; footprint Connector_JST:JST_PH_B5B-PH-K_1x05_P2.00mm_Vertical -> Connector_JST:JST_PH_B6B-PH-K_1x06_P2.00mm_Vertical
- moved D102 65.1 mm to (148.3, 56.7)
- moved D107 65.1 mm to (148.3, 55.2)
- moved R107 64.3 mm to (148.8, 64.0), turned to 180 degrees
- moved R108 61.5 mm to (147.0, 64.0), turned to 0 degrees
- moved D105 60.6 mm to (145.2, 63.6), turned to -90 degrees
- moved C105 60.3 mm to (143.3, 63.6), turned to 0 degrees
- moved D106 59.8 mm to (144.6, 63.6), turned to -90 degrees
- moved U101 59.4 mm to (140.7, 64.3), turned to -90 degrees
- moved U102 58.5 mm to (103.9, 67.1)
- moved J102 55.7 mm to (147.2, 69.8)
- moved C103 55.5 mm to (141.8, 68.3), turned to 90 degrees
- moved R109 53.4 mm to (140.7, 68.3), turned to -90 degrees
- moved C111 52.7 mm to (139.5, 68.3), turned to 90 degrees
- moved C104 50.7 mm to (140.7, 66.6), turned to 180 degrees
- moved J101 49.4 mm to (141.6, 59.7), turned to 0 degrees
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Connections:
- C203 pad 1: Net-(U201-CPL) -> Net-(U201-CPH)
- C203 pad 2: Net-(U201-CPH) -> Net-(U201-CPL)
- C205 pad 1: /Motor Driver 1/VREF -> +3.3V
- C208 pad 1: Net-(U202-CPL) -> Net-(U202-CPH)
- C208 pad 2: Net-(U202-CPH) -> Net-(U202-CPL)
- C209 pad 1: /Motor Driver 2/VREF -> +3.3V
- J103 pad 1: /sns_miso -> /sns_mosi
- J103 pad 2: /sns_mosi -> /sns_miso
- J103 pad 3: /sns_cs2 -> /sns_sck
- J103 pad 4: +3.3V -> /sns_cs2
- J103 pad 5: GND -> +3.3V
- R211 pad 2: 3.3V -> +3.3V
- R222 pad 2: 3.3V -> +3.3V
- U103 pad 10: /snsB1 -> /CHC1
- U103 pad 11: /snsA1 -> /CHB1
- U103 pad 12: /CAL1 -> /CHA1
- U103 pad 15: /sns_sck -> /snsA1
- U103 pad 17: /sns_cs1 -> /snsB1
- U103 pad 18: /CHB1 -> /snsC1
- U103 pad 20: /ctrl_scl -> /FAULT1
- U103 pad 21: /ctrl_sda -> /sns_cs1
- U103 pad 23: /sns_cs2 -> /sns_sck
- U103 pad 35: /CHA1 -> /sns_cs2
- U103 pad 38: /snsB2 -> /snsA2
- U103 pad 39: /snsA2 -> /snsB2
- U103 pad 4: /snsC1 -> unconnected-(U103-IO4-Pad4)
- U103 pad 6: /CHC1 -> /EN1
- U103 pad 7: /FAULT1 -> /CAL1
- U103 pad 8: /EN1 -> /ctrl_sda
- U103 pad 9: unconnected-(U103-IO16-Pad9) -> /ctrl_scl
- U201 pad 24: /Motor Driver 1/VREF -> +3.3V
- U202 pad 24: /Motor Driver 2/VREF -> +3.3V
Routing:
- net +3.3V: track 0.00 -> 99.1 mm, vias 0 -> 4
- net M+: track 1.23 -> 45.5 mm, vias 106 -> 120
- net /sns_cs1: track 0.00 -> 35.0 mm, vias 0 -> 1
- net /sns_sck: track 0.00 -> 22.5 mm, vias 0 -> 1
- net /sns_cs2: track 0.00 -> 21.6 mm
- net /sns_miso: track 0.00 -> 20.0 mm, vias 0 -> 1
- net /sns_mosi: track 0.00 -> 17.5 mm, vias 0 -> 1
- net /D-: track 5.04 -> 21.9 mm, vias 1 -> 3
- net /D+: track 4.73 -> 20.7 mm, vias 1 -> 3
- net /EN1: track 1.09 -> 16.2 mm
- net /snsC1: track 0.00 -> 14.4 mm, vias 0 -> 2
- net /snsB1: track 0.00 -> 13.6 mm, vias 0 -> 2
- net +5V: track 0.00 -> 13.2 mm
- net /CAL1: track 3.16 -> 14.2 mm
- net /CHC1: track 1.29 -> 12.3 mm, vias 0 -> 2
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- removed copper zone on F.Cu, net +5V

Commit message: finished iteration 1
Parts:
- removed J102: USB_C_Receptacle_USB2.0_14P, Connector_USB:USB_C_Receptacle_HCTL_HC-TYPE-C-16P-01A
- removed Q102, Q103, Q104, Q105, Q106, Q303, Q403, Q503: AGM6014AP, easyeda2kicad:PDFN-8_L3.1-W3.0-P0.65-LS3.3-BL
- removed R224: 47k, Resistor_SMD:R_0402_1005Metric
- removed U102: XT60H-M, easyeda2kicad:CONN-TH_XT60H-M
- added C102: 4.7u, Capacitor_SMD:C_0402_1005Metric, F.Cu at (148.4, 55.4)
- added C106: 100n, Capacitor_SMD:C_0402_1005Metric, F.Cu at (125.1, 63.6)
- added C107: 100n, Capacitor_SMD:C_0402_1005Metric, F.Cu at (122.0, 71.3)
- added C112: 1u, Capacitor_SMD:C_0402_1005Metric, F.Cu at (145.2, 59.0)
- added C113: 100n, Capacitor_SMD:C_0402_1005Metric, F.Cu at (122.9, 63.9)
- added C114: 1u, Capacitor_SMD:C_0402_1005Metric, F.Cu at (121.9, 63.9)
- added C115: 4.7u, Capacitor_SMD:C_0402_1005Metric, F.Cu at (127.1, 63.6)
- added C116: 220n, Capacitor_SMD:C_0402_1005Metric, F.Cu at (135.4, 73.7)
- added CN101: XT60PB-F.G.Y, easyeda2kicad:CONN-TH_XT60PB-F.G.Y, F.Cu at (103.9, 67.1)
- added D103: H5VL10B, easyeda2kicad:SOD-882_L1.0-W0.6-BI, F.Cu at (144.8, 66.5)
- added D104: 1N5819WS, Diode_SMD:D_SOD-323, F.Cu at (137.6, 71.6)
- added H101: MountingHole, easyeda2kicad:JLC_Tooling_Hole, F.Cu at (125.0, 26.4)
- added H102: MountingHole, easyeda2kicad:JLC_Tooling_Hole, F.Cu at (148.8, 26.2)
- added H103: MountingHole, easyeda2kicad:JLC_Tooling_Hole, F.Cu at (112.0, 65.5)
- added H104: MountingHole, easyeda2kicad:JLC_Tooling_Hole, F.Cu at (101.2, 26.2)
- added H105: MountingHole, MountingHole:MountingHole_2.2mm_M2, F.Cu at (125.0, 32.0)
- added H106: MountingHole, MountingHole:MountingHole_2.2mm_M2, F.Cu at (125.0, 42.0)
- added H107: MountingHole, easyeda2kicad:JLC_Tooling_Hole, F.Cu at (148.7, 49.8)
- added J105: USB-TYPE-C-019, easyeda2kicad:TYPE-C-SMD_HX-TYPE-C-16PIN, F.Cu at (144.3, 70.9)
- added Q302: XRS100N06LD, easyeda2kicad:DFN-8_L3.0-W3.0-P0.65-BL-4, F.Cu at (144.2, 37.7)
- added Q402: XRS100N06LD, easyeda2kicad:DFN-8_L3.0-W3.0-P0.65-BL-4, F.Cu at (137.0, 37.7)
- added Q502: XRS100N06LD, easyeda2kicad:DFN-8_L3.0-W3.0-P0.65-BL-4, F.Cu at (129.6, 37.7)
- added Q701: XRS100N06LD, easyeda2kicad:DFN-8_L3.0-W3.0-P0.65-BL-4, F.Cu at (116.8, 37.4)
- added Q702: XRS100N06LD, easyeda2kicad:DFN-8_L3.0-W3.0-P0.65-BL-4, F.Cu at (120.5, 37.4)
- added Q801: XRS100N06LD, easyeda2kicad:DFN-8_L3.0-W3.0-P0.65-BL-4, F.Cu at (102.2, 37.4)
- added Q802: XRS100N06LD, easyeda2kicad:DFN-8_L3.0-W3.0-P0.65-BL-4, F.Cu at (105.8, 37.4)
- added Q901: XRS100N06LD, easyeda2kicad:DFN-8_L3.0-W3.0-P0.65-BL-4, F.Cu at (109.6, 37.4)
- added Q902: XRS100N06LD, easyeda2kicad:DFN-8_L3.0-W3.0-P0.65-BL-4, F.Cu at (113.3, 37.4)
- added R112: 100k, Resistor_SMD:R_0402_1005Metric, F.Cu at (146.4, 61.2)
- added R113: 3.3k, PCM_SparkFun-Resistor:R_0402_1005Metric, F.Cu at (144.4, 61.2)
- added R114: 330, Resistor_SMD:R_0402_1005Metric, F.Cu at (136.0, 71.5)
- added R207: 100k, Resistor_SMD:R_0402_1005Metric, F.Cu at (140.2, 58.2)
- added R208: 100k, Resistor_SMD:R_0402_1005Metric, F.Cu at (143.0, 57.3)
- added R604: 100k, Resistor_SMD:R_0402_1005Metric, F.Cu at (117.3, 57.0)
- added SW102: TS-1088-AR02016, easyeda2kicad:SW-SMD_L3.9-W3.0-P4.45, F.Cu at (141.5, 63.4)
- C104: value 22u -> 100n; footprint Capacitor_SMD:C_0603_1608Metric -> Capacitor_SMD:C_0402_1005Metric
- C111: value 1u -> 10n
- C201, C206: footprint Capacitor_SMD:C_0805_2012Metric -> Capacitor_SMD:C_0402_1005Metric
- C205, C209: value 0.1u -> 100n
- D102, D107: value B16WS_C7420327 -> 1N5819WS; footprint easyeda2kicad:SOD-323_L1.7-W1.3-LS2.5-FD -> Diode_SMD:D_SOD-323
- D105: value H5VL06B -> H5VL10B; footprint easyeda2kicad:X3-DFN0603-2_L0.6-W0.3-BI -> easyeda2kicad:SOD-882_L1.0-W0.6-BI
- D106: value H5VL06B -> LED; footprint easyeda2kicad:X3-DFN0603-2_L0.6-W0.3-BI -> LED_SMD:LED_0603_1608Metric
- Q101: value AGM6014AP -> AO3400A; footprint easyeda2kicad:PDFN-8_L3.1-W3.0-P0.65-LS3.3-BL -> easyeda2kicad:SOT-23-3_L2.9-W1.3-P1.90-LS2.4-BR
- Q301, Q401, Q501: value AGM6014AP -> XRS100N06LD; footprint easyeda2kicad:PDFN-8_L3.1-W3.0-P0.65-LS3.3-BL -> easyeda2kicad:DFN-8_L3.0-W3.0-P0.65-BL-4
- R109: value 10k -> 3.3k
- R602: value 47k -> 100k
- U103: value ESP32-S3-WROOM-1 -> STM32G474CBTx; footprint RF_Module:ESP32-S3-WROOM-1 -> Package_QFP:LQFP-48_7x7mm_P0.5mm
- moved D107 42.9 mm to (109.4, 73.2), turned to -90 degrees
- moved Q101 38.6 mm to (145.4, 63.4)
- moved J101 30.9 mm to (113.0, 71.4)
- moved R222 25.8 mm to (122.0, 73.2), turned to 90 degrees
- moved R211 20.5 mm to (133.8, 71.5), turned to -90 degrees
- moved R110 16.2 mm to (122.2, 49.8), turned to 0 degrees
- moved R111 15.1 mm to (122.2, 50.8)
- moved J103 14.9 mm to (123.1, 53.5), turned to 0 degrees
- moved C104 11.0 mm to (132.2, 73.7), turned to 0 degrees
- moved D106 10.1 mm to (136.0, 69.0)
- moved D102 9.65 mm to (148.1, 66.4), turned to 0 degrees
- moved C103 9.51 mm to (133.8, 73.4), turned to -90 degrees
- moved SW101 9.06 mm to (137.7, 63.4)
- moved U101 8.94 mm to (147.9, 59.0), turned to 180 degrees
- moved U104 8.68 mm to (148.1, 64.7), turned to 180 degrees
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Connections:
- C205 pad 1: +3.3V -> /VREF
- C209 pad 1: +3.3V -> /VREF
- D102 pad 1: Net-(D102-A) -> +5V
- D102 pad 2: +5V -> Net-(D102-A)
- D106 pad 2: /D+ -> Net-(D106-A)
- D107 pad 1: Net-(D107-A) -> +5V
- D107 pad 2: +5V -> Net-(D107-A)
- J101 pad 1: /ctrl_scl -> GND
- J101 pad 2: /ctrl_sda -> Net-(D107-A)
- J101 pad 3: GND -> /ctrl_sda
- J101 pad 4: Net-(D107-A) -> /ctrl_scl
- Q101 pad 1: /Motor Driver 2/Pole 1/PoleOut -> Net-(D104-A)
- Q101 pad 2: /Motor Driver 2/Pole 1/PoleOut -> GND
- Q101 pad 3: /Motor Driver 2/Pole 1/PoleOut -> /~{rst}
- Q301 pad 1: /Motor Driver 1/Pole 1/PoleOut -> /Motor Driver 1/Pole 1/SP
- Q301 pad 2: /Motor Driver 1/Pole 1/PoleOut -> /Motor Driver 1/Pole 1/SP
- Q301 pad 3: /Motor Driver 1/Pole 1/PoleOut -> /Motor Driver 1/Pole 1/SP
- Q301 pad 4: /Motor Driver 1/Pole 1/GH -> /Motor Driver 1/Pole 1/GL
- Q301 pad 5: M+ -> /Motor Driver 1/Pole 1/PoleOut
- Q401 pad 1: /Motor Driver 1/Pole 2/PoleOut -> /Motor Driver 1/Pole 2/SP
- Q401 pad 2: /Motor Driver 1/Pole 2/PoleOut -> /Motor Driver 1/Pole 2/SP
- Q401 pad 3: /Motor Driver 1/Pole 2/PoleOut -> /Motor Driver 1/Pole 2/SP
- Q401 pad 4: /Motor Driver 1/Pole 2/GH -> /Motor Driver 1/Pole 2/GL
- Q401 pad 5: M+ -> /Motor Driver 1/Pole 2/PoleOut
- Q501 pad 1: /Motor Driver 1/Pole 3/PoleOut -> /Motor Driver 1/Pole 3/SP
- Q501 pad 2: /Motor Driver 1/Pole 3/PoleOut -> /Motor Driver 1/Pole 3/SP
- Q501 pad 3: /Motor Driver 1/Pole 3/PoleOut -> /Motor Driver 1/Pole 3/SP
- Q501 pad 4: /Motor Driver 1/Pole 3/GH -> /Motor Driver 1/Pole 3/GL
- Q501 pad 5: M+ -> /Motor Driver 1/Pole 3/PoleOut
- R109 pad 1: +3.3V -> /CHLB2
- R109 pad 2: /~{rst} -> Net-(D104-K)
- R206 pad 1: /Motor Driver 1/~{HI-Z} -> /CHLA1
- R602 pad 1: Net-(U202-MODE) -> /CHLA2
- R603 pad 1: /~{HI-Z2} -> /CHLB2
- SW101 pad 1: /~{rst} -> GND
- SW101 pad 2: GND -> /~{rst}
- U103 pad 1: GND -> +3.3V
- U103 pad 10: /CHC1 -> /snsC1
- U103 pad 11: /CHB1 -> /CAL1
- U103 pad 12: /CHA1 -> /EN1
- U103 pad 13: /D- -> /sns_sck
- U103 pad 14: /D+ -> /sns_miso
- U103 pad 15: /snsA1 -> /sns_mosi
- U103 pad 16: unconnected-(U103-IO46-Pad16) -> /CHB1
- U103 pad 17: /snsB1 -> /CHLC2
- U103 pad 18: /snsC1 -> /sns_cs2
- U103 pad 19: /GAIN1 -> GND
- U103 pad 2: +3.3V -> /CHLA1
- U103 pad 20: /FAULT1 -> /VREF
- U103 pad 21: /sns_cs1 -> +3.3V
- U103 pad 22: /snsC2 -> /sns_cs1
- U103 pad 23: /sns_sck -> GND
- U103 pad 24: /sns_miso -> +3.3V
- U103 pad 25: /sns_mosi -> /CAL2
- U103 pad 26: unconnected-(U103-IO45-Pad26) -> /snsB2
- U103 pad 27: unconnected-(U103-IO0-Pad27) -> /EN2
- U103 pad 28: /CHC2 -> /snsA2
- U103 pad 29: /CHB2 -> /snsC2
- U103 pad 3: /~{rst} -> /FAULT1
- U103 pad 30: /CHA2 -> /CHA1
- U103 pad 31: /CAL2 -> /CHLB1
- U103 pad 32: /EN2 -> /CHC1
- U103 pad 33: /GAIN2 -> /D-
- U103 pad 34: /FAULT2 -> /D+
- U103 pad 35: /sns_cs2 -> GND
- U103 pad 36: unconnected-(U103-RXD0-Pad36) -> +3.3V
- U103 pad 37: unconnected-(U103-TXD0-Pad37) -> /ctrl_scl
- U103 pad 38: /snsA2 -> /ctrl_sda
- U103 pad 39: /snsB2 -> /FAULT2
- U103 pad 4: unconnected-(U103-IO4-Pad4) -> /GAIN1
- U103 pad 40: GND -> /CHA2
- U103 pad 41: GND -> /CHB2
- U103 pad 5: unconnected-(U103-IO5-Pad5) -> /CHLC1
- U103 pad 6: /EN1 -> unconnected-(U103-PF1-Pad6)
- U103 pad 7: /CAL1 -> /~{rst}
- U103 pad 8: /ctrl_sda -> /snsA1
- U103 pad 9: /ctrl_scl -> /snsB1
- U201 pad 24: +3.3V -> /VREF
- U201 pad 26: Net-(U201-MODE) -> GND
- U201 pad 35: /Motor Driver 1/~{HI-Z} -> /CHLA1
- U201 pad 37: /Motor Driver 1/~{HI-Z} -> /CHLB1
- U201 pad 39: /Motor Driver 1/~{HI-Z} -> /CHLC1
- U202 pad 24: +3.3V -> /VREF
- U202 pad 26: Net-(U202-MODE) -> GND
- U202 pad 35: /~{HI-Z2} -> /CHLA2
- U202 pad 37: /~{HI-Z2} -> /CHLB2
- U202 pad 39: /~{HI-Z2} -> /CHLC2
Routing:
- net /VREF: track 0.00 -> 55.7 mm, vias 0 -> 4
- net +5V: track 13.2 -> 57.0 mm, vias 0 -> 2
- net /CHLB2: track 0.00 -> 37.0 mm, vias 0 -> 2
- net /CHLA2: track 0.00 -> 29.8 mm, vias 0 -> 2
- net /CHLB1: track 0.00 -> 26.1 mm, vias 0 -> 2
- net /CHLA1: track 0.00 -> 22.8 mm, vias 0 -> 2
- net /CHLC1: track 0.00 -> 22.1 mm, vias 0 -> 2
- net /CHC2: track 7.77 -> 26.9 mm, vias 0 -> 2
- net /CHLC2: track 0.00 -> 19.1 mm
- net /CHA2: track 12.0 -> 29.2 mm, vias 0 -> 2
- net /Motor Driver 2/Pole 1/GL: track 40.5 -> 23.3 mm
- net /CHA1: track 7.36 -> 23.5 mm, vias 0 -> 2
- net +3.3V: track 99.1 -> 83.1 mm, vias 4 -> 5
- net /FAULT1: track 11.3 -> 27.2 mm
- net /CHB2: track 10.4 -> 26.1 mm, vias 0 -> 2
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- added copper zone on F.Cu, net +3.3V
- added copper zone on F.Cu, net /VREF
Other:
- board text added: "+"
- board text added: "-"
- board text added: "36V MAX"
- board text added: "GND 5V SDA SCL"
- board text added: "I2C"
- board text added: "MOSI MISO SCK CS 3.3V GND"
- board text added: "PROG"
- board text added: "RST"
- board text added: "SPI"
- board text added: "V1"

Commit message: generated production files
Parts:
- moved D104 0.24 mm to (137.8, 71.5), turned to 90 degrees
- moved R108 0.13 mm to (145.9, 66.3)
- turned D102 to 180 degrees
- turned D107 to 90 degrees
